File: PCB/LegoRCHub_8ch/LegoRCHub_8ch.kicad_pcb (KiCad board)
At the start: 2 copper layers, 39.3 x 55.2 mm, 35 parts, among them J1 Conn_01x02, J10 Conn_01x02, J11 Conn_01x03, J2 Conn_01x02, J3 Conn_01x02, J4 Conn_01x02, J5 Conn_01x03, J6 Conn_01x03, J7 Conn_01x03, J8 Conn_01x03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

Commit message: ...
Connections:
- net Net-(U7-Pad11) renamed /LED
Routing:
- net GND: vias 45 -> 46
- net (no net): vias 1 -> 0
Changed lines of the file:
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@@
   (net 32 "unconnected-(U7-Pad7)")
   (net 33 "unconnected-(U7-Pad6)")
-  (net 34 "Net-(U7-Pad11)")
+  (net 34 "/LED")
   (footprint "Capacitor_SMD:C_1206_3216Metric_Pad1.33x1.80mm_HandSolder" (layer "F.Cu")
     (at 57.45 66.8)
@@
       (net 19 "/CH4_3") (pinfunction "PB1") (pintype "bidirectional"))
     (pad "11" smd roundrect (at 3.5 -2.925 180) (size 1.9 0.5) (layers "B.Cu" "B.Paste" "B.Mask") (roundrect_rratio 0.25)
-      (net 34 "Net-(U7-Pad11)") (pinfunction "PB0") (pintype "bidirectional"))
+      (net 34 "/LED") (pinfunction "PB0") (pintype "bidirectional"))
     (pad "12" smd roundrect (at 3.5 -2.275 180) (size 1.9 0.5) (layers "B.Cu" "B.Paste" "B.Mask") (roundrect_rratio 0.25)
       (net 25 "unconnected-(U7-Pad12)") (pinfunction "PC0") (pintype "bidirectional+no_connect"))
@@
       (net 31 "Net-(D1-Pad1)") (pinfunction "K") (pintype "passive"))
     (pad "2" smd roundrect (at 1.025 0 180) (size 1.15 1.4) (layers "B.Cu" "B.Paste" "B.Mask") (roundrect_rratio 0.2173913043)
-      (net 34 "Net-(U7-Pad11)") (pinfunction "A") (pintype "passive"))
+      (net 34 "/LED") (pinfunction "A") (pintype "passive"))
     (model "${KICAD6_3DMODEL_DIR}/LED_SMD.3dshapes/LED_0805_2012Metric.wrl"
       (offset (xyz 0 0 0))
@@
   (gr_line locked (start 64.08 74.71) (end 64.08 26.89) (layer "Edge.Cuts") (width 0.15))
   (gr_arc locked (start 24.82 26.89) (mid 25.900776 24.280776) (end 28.51 23.2) (layer "Edge.Cuts") (width 0.15))
-  (via (at 36.45 54.8) (size 0.8) (drill 0.4) (layers "F.Cu" "B.Cu") (free) (net 0))
   (segment (start 31.075 65.435) (end 32.665 65.435) (width 0.25) (layer "F.Cu") (net 1))
   (segment (start 57.825 36.165) (end 56.235 36.165) (width 0.25) (layer "F.Cu") (net 1))
@@
   (via (at 54.45 32.8) (size 0.8) (drill 0.4) (layers "F.Cu" "B.Cu") (free) (net 1))
   (via (at 52.45 44.8) (size 0.8) (drill 0.4) (layers "F.Cu" "B.Cu") (free) (net 1))
+  (via (at 36.45 54.8) (size 0.8) (drill 0.4) (layers "F.Cu" "B.Cu") (free) (net 1))
   (via (at 36.45 60.8) (size 0.8) (drill 0.4) (layers "F.Cu" "B.Cu") (free) (net 1))
   (via (at 38.45 70.8) (size 0.8) (drill 0.4) (layers "F.Cu" "B.Cu") (free) (net 1))

Commit message: LegoRCHub_8ch: beta 8 (layout somewhat finished)
Parts:
- C1, C3, C5, C7: value 47uF -> 100uF
- J11: value Conn_01x03 -> Conn_01x03_MountingPin; footprint Connector_JST:JST_XH_B3B-XH-A_1x03_P2.50mm_Vertical -> Connector_JST:JST_SH_BM03B-SRSS-TB_1x03-1MP_P1.00mm_Vertical
- U6: value AMS1117-5.0 -> L78L05_SOT89; footprint Package_TO_SOT_SMD:SOT-89-3_Handsoldering -> Package_TO_SOT_SMD:SOT-89-3
- moved J11 7.43 mm to (44.5, 63.3)
- moved J10 5.00 mm to (45.7, 69.3)
- moved U6 0.94 mm to (43.2, 40.4)
Connections:
- U6 pad 1: GND -> VCC
- U6 pad 2: VCC -> GND
Routing:
- net /IBus: track 21.9 -> 11.4 mm, vias 1 -> 0
- net VCC: track 36.9 -> 42.4 mm, vias 1 -> 2
- net /UPDI: track 15.9 -> 21.1 mm
- net +BATT: track 11.3 -> 16.2 mm
- net /CH6: track 9.96 -> 10.6 mm
- net GND: vias 46 -> 85
- removed copper zone on B.Cu, net VCC
Other:
- board text added: "+"
- board text added: "-"
- board text added: "13V MAX"
- board text added: "CH1"
- board text added: "CH2"
- board text added: "CH3"
- board text added: "CH4"
- board text added: "CH5"
- board text added: "CH6"
- board text added: "CH7"
- board text added: "CH8"
- board text added: "D"
- board text added: "RX"
- board text added: "UPDI"
