File: PCB/LegoRCHub_8ch/LegoRCHub_8ch.kicad_sch (KiCad schematic)
At the start: 31 parts, among them J1 Conn_01x02, J10 Conn_01x02, J11 Conn_01x03, J2 Conn_01x02, J3 Conn_01x02, J4 Conn_01x02, J5 Conn_01x03, J6 Conn_01x03, J7 Conn_01x03, J8 Conn_01x03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

Commit message: LegoRCHub_8ch: beta 8 (layout somewhat finished)
Parts:
- removed J11: Conn_01x03, Connector_JST:JST_XH_B3B-XH-A_1x03_P2.50mm_Vertical, symbol Connector_Generic:Conn_01x03
- removed U6: AMS1117-5.0, Package_TO_SOT_SMD:SOT-89-3_Handsoldering, symbol Regulator_Linear:AMS1117-5.0
- added J11: Conn_01x03_MountingPin, Connector_JST:JST_SH_BM03B-SRSS-TB_1x03-1MP_P1.00mm_Vertical, symbol Connector_Generic_MountingPin:Conn_01x03_MountingPin
- added U6: L78L05_SOT89, Package_TO_SOT_SMD:SOT-89-3, symbol Regulator_Linear:L78L05_SOT89
- C1, C3, C5, C7: value 47uF -> 100uF
Connections:
- net +BATT: now also U6.3 (IN)
- net GND: now also J11.1 (Pin_1), J11.MP (MountPin), U6.2 (GND)
- net IBus: now also J11.3 (Pin_3)
- net VCC: now also J11.2 (Pin_2), U6.1 (OUT)
- no-connect marks 3 -> 7
