File: PCB/LegoRCHub_10ch/LegoRCHub_10ch.kicad_sch (KiCad schematic)
At the start: 37 parts, among them J1 Conn_01x02, J10 Conn_01x03, J11 Conn_01x03_MountingPin, J12 Conn_01x02, J13 Conn_01x02, J2 Conn_01x02, J3 Conn_01x02, J4 Conn_01x02, J5 Conn_01x02, J6 Conn_01x02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

Commit message: LegoRCHub_10ch: ...
Connections:
- net CH10: no longer U7.9 (PB2)
- net CH1_2: now also U7.3 (PA5); no longer U7.18 (PA2)
- net CH1_3: now also U7.2 (PA4); no longer U7.19 (PA3)
- net CH2_2: no longer U7.2 (PA4)
- net CH2_3: no longer U7.3 (PA5)
- net CH3_2: now also U7.5 (PA7); no longer U7.15 (PC3)
- net CH3_3: now also U7.4 (PA6); no longer U7.17 (PA1)
- net CH4_2: now also U7.19 (PA3); no longer U7.4 (PA6)
- net CH4_3: now also U7.18 (PA2); no longer U7.5 (PA7)
- net CH5_2: now also U7.10 (PB1); no longer U7.13 (PC1)
- net CH5_3: now also U7.9 (PB2); no longer U7.14 (PC2)
- net CH6_2: now also U7.17 (PA1); no longer U7.6 (PB5)
- net CH6_3: now also U7.11 (PB0); no longer U7.7 (PB4)
- net CH7: no longer U7.12 (PC0)
- net CH8: no longer U7.11 (PB0)
- net CH9: no longer U7.10 (PB1)
Changed lines of the file:
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@@
     (effects (font (size 1.27 1.27)) (justify right bottom))
   )
-  (label "CH5_3" (at 163.83 97.79 180)
-    (effects (font (size 1.27 1.27)) (justify right bottom))
+  (label "CH5_3" (at 194.31 97.79 0)
+    (effects (font (size 1.27 1.27)) (justify left bottom))
   )
   (label "CH9" (at 80.01 187.325 270)
@@
     (effects (font (size 1.27 1.27)) (justify right bottom))
   )
-  (label "CH1_2" (at 194.31 74.93 0)
+  (label "CH1_2" (at 194.31 82.55 0)
     (effects (font (size 1.27 1.27)) (justify left bottom))
   )
-  (label "CH3_2" (at 163.83 100.33 180)
-    (effects (font (size 1.27 1.27)) (justify right bottom))
+  (label "CH3_2" (at 194.31 87.63 0)
+    (effects (font (size 1.27 1.27)) (justify left bottom))
   )
-  (label "CH7" (at 163.83 92.71 180)
+  (label "CH7" (at 236.22 71.12 180)
     (effects (font (size 1.27 1.27)) (justify right bottom))
   )
@@
     (effects (font (size 1.27 1.27)) (justify right bottom))
   )
-  (label "CH8" (at 194.31 92.71 0)
+  (label "CH8" (at 245.11 91.44 0)
     (effects (font (size 1.27 1.27)) (justify left bottom))
   )
@@
     (effects (font (size 1.27 1.27)) (justify right bottom))
   )
-  (label "CH3_3" (at 194.31 72.39 0)
+  (label "CH3_3" (at 194.31 85.09 0)
     (effects (font (size 1.27 1.27)) (justify left bottom))
   )
-  (label "CH9" (at 194.31 95.25 0)
+  (label "CH9" (at 245.11 93.98 0)
     (effects (font (size 1.27 1.27)) (justify left bottom))
   )
-  (label "CH5_2" (at 163.83 95.25 180)
-    (effects (font (size 1.27 1.27)) (justify right bottom))
+  (label "CH5_2" (at 194.31 95.25 0)
+    (effects (font (size 1.27 1.27)) (justify left bottom))
   )
   (label "CH4_3" (at 96.52 96.52 180)
@@
     (effects (font (size 1.27 1.27)) (justify right bottom))
   )
-  (label "CH1_3" (at 194.31 77.47 0)
+  (label "CH1_3" (at 194.31 80.01 0)
     (effects (font (size 1.27 1.27)) (justify left bottom))
   )
-  (label "CH2_2" (at 194.31 80.01 0)
+  (label "CH2_2" (at 218.44 102.87 0)
     (effects (font (size 1.27 1.27)) (justify left bottom))
   )
@@
     (effects (font (size 1.27 1.27)) (justify right bottom))
   )
-  (label "CH10" (at 194.31 97.79 0)
+  (label "CH10" (at 245.11 96.52 0)
     (effects (font (size 1.27 1.27)) (justify left bottom))
   )
-  (label "CH4_3" (at 194.31 87.63 0)
+  (label "CH4_3" (at 194.31 74.93 0)
     (effects (font (size 1.27 1.27)) (justify left bottom))
   )
@@
     (effects (font (size 1.27 1.27)) (justify right bottom))
   )
-  (label "CH6_2" (at 194.31 105.41 0)
+  (label "CH6_2" (at 194.31 72.39 0)
     (effects (font (size 1.27 1.27)) (justify left bottom))
   )
-  (label "CH6_3" (at 194.31 102.87 0)
+  (label "CH6_3" (at 194.31 92.71 0)
     (effects (font (size 1.27 1.27)) (justify left bottom))
   )
@@
     (effects (font (size 1.27 1.27)) (justify right bottom))
   )
-  (label "CH4_2" (at 194.31 85.09 0)
+  (label "CH4_2" (at 194.31 77.47 0)
     (effects (font (size 1.27 1.27)) (justify left bottom))
   )
-  (label "CH2_3" (at 194.31 82.55 0)
+  (label "CH2_3" (at 218.44 105.41 0)
     (effects (font (size 1.27 1.27)) (justify left bottom))
   )

Commit message: LegoRCHub_10ch: improved design - beta 1
Parts:
- removed J12: Conn_01x02, Connector_PinSocket_2.54mm:PinSocket_1x02_P2.54mm_Vertical, symbol Connector_Generic:Conn_01x02
- added J13: Conn_01x01, Connector_Wire:SolderWirePad_1x01_SMD_1x2mm, symbol Connector_Generic:Conn_01x01
- renumbered J13 to J12
Connections:
- net CH10: now also U7.13 (PC1)
- net CH2_2: now also U7.6 (PB5)
- net CH2_3: now also U7.7 (PB4)
- net CH7: now also U7.15 (PC3)
- net CH8: now also U7.12 (PC0)
- net CH9: now also U7.14 (PC2)
- net UPDI: now also J13.1 (Pin_1)
Changed lines of the file:
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@@
     (effects (font (size 1.27 1.27)) (justify left bottom))
   )
-  (label "CH7" (at 236.22 71.12 180)
+  (label "CH7" (at 163.83 100.33 180)
     (effects (font (size 1.27 1.27)) (justify right bottom))
   )
@@
     (effects (font (size 1.27 1.27)) (justify right bottom))
   )
-  (label "CH8" (at 245.11 91.44 0)
-    (effects (font (size 1.27 1.27)) (justify left bottom))
+  (label "CH8" (at 163.83 92.71 180)
+    (effects (font (size 1.27 1.27)) (justify right bottom))
   )
   (label "CH6_3" (at 95.25 148.59 180)
@@
     (effects (font (size 1.27 1.27)) (justify left bottom))
   )
-  (label "CH9" (at 245.11 93.98 0)
-    (effects (font (size 1.27 1.27)) (justify left bottom))
+  (label "CH9" (at 163.83 97.79 180)
+    (effects (font (size 1.27 1.27)) (justify right bottom))
   )
   (label "CH5_2" (at 194.31 95.25 0)
@@
     (effects (font (size 1.27 1.27)) (justify left bottom))
   )
-  (label "CH2_2" (at 218.44 102.87 0)
+  (label "CH2_2" (at 194.31 105.41 0)
     (effects (font (size 1.27 1.27)) (justify left bottom))
   )
-  (label "UPDI" (at 170.18 132.08 180)
+  (label "UPDI" (at 170.18 129.54 180)
     (effects (font (size 1.27 1.27)) (justify right bottom))
   )
-  (label "CH10" (at 245.11 96.52 0)
-    (effects (font (size 1.27 1.27)) (justify left bottom))
+  (label "CH10" (at 163.83 95.25 180)
+    (effects (font (size 1.27 1.27)) (justify right bottom))
   )
   (label "CH4_3" (at 194.31 74.93 0)
@@
     (effects (font (size 1.27 1.27)) (justify left bottom))
   )
-  (label "CH2_3" (at 218.44 105.41 0)
+  (label "CH2_3" (at 194.31 102.87 0)
     (effects (font (size 1.27 1.27)) (justify left bottom))
   )
@@
     (pin "1")
   )
+  (symbol (lib_id "Connector_Generic:Conn_01x01") (at 175.26 129.54 0) (unit 1)
+    (in_bom yes) (on_board yes) (fields_autoplaced)
+    (property "Reference" "J13" (id 0) (at 177.8 128.2699 0)
+      (effects (font (size 1.27 1.27)) (justify left))
+    )
+    (property "Value" "Conn_01x01" (id 1) (at 177.8 130.8099 0)
+      (effects (font (size 1.27 1.27)) (justify left))
+    )
+    (property "Footprint" "Connector_Wire:SolderWirePad_1x01_SMD_1x2mm" (id 2) (at 175.26 129.54 0)
+      (effects (font (size 1.27 1.27)) hide)
+    )
+    (property "Datasheet" "~" (id 3) (at 175.26 129.54 0)
+      (effects (font (size 1.27 1.27)) hide)
+    )
+    (pin "1")
+  )
   (symbol (lib_id "power:VCC") (at 170.18 143.51 90) (unit 1)
     (in_bom yes) (on_board yes) (fields_autoplaced)
@@
     )
     (pin "1")
-  )
-  (symbol (lib_id "Connector_Generic:Conn_01x02") (at 175.26 129.54 0) (unit 1)
-    (in_bom yes) (on_board yes) (fields_autoplaced)
-    (property "Reference" "J12" (id 0) (at 177.8 129.5399 0)
-      (effects (font (size 1.27 1.27)) (justify left))
-    )
-    (property "Value" "Conn_01x02" (id 1) (at 177.8 132.0799 0)
-      (effects (font (size 1.27 1.27)) (justify left))
-    )
-    (property "Footprint" "Connector_PinSocket_2.54mm:PinSocket_1x02_P2.54mm_Vertical" (id 2) (at 175.26 129.54 0)
-      (effects (font (size 1.27 1.27)) hide)
-    )
-    (property "Datasheet" "~" (id 3) (at 175.26 129.54 0)
-      (effects (font (size 1.27 1.27)) hide)
-    )
-    (pin "1")
-    (pin "2")
   )
   (symbol (lib_id "Connector_Generic:Conn_01x02") (at 58.42 146.05 0) (unit 1)
@@
   (symbol (lib_id "Connector_Generic:Conn_01x02") (at 254 41.91 0) (unit 1)
     (in_bom yes) (on_board yes) (fields_autoplaced)
-    (property "Reference" "J13" (id 0) (at 256.54 41.9099 0)
+    (property "Reference" "J12" (id 0) (at 256.54 41.9099 0)
       (effects (font (size 1.27 1.27)) (justify left))
     )
@@
     (pin "2")
   )
-  (symbol (lib_id "power:GND") (at 170.18 129.54 270) (unit 1)
-    (in_bom yes) (on_board yes) (fields_autoplaced)
-    (property "Reference" "#PWR042" (id 0) (at 163.83 129.54 0)
-      (effects (font (size 1.27 1.27)) hide)
-    )
-    (property "Value" "GND" (id 1) (at 171.45 129.5399 90)
-      (effects (font (size 1.27 1.27)) (justify left))
-    )
-    (property "Footprint" "" (id 2) (at 170.18 129.54 0)
-      (effects (font (size 1.27 1.27)) hide)
-    )
-    (property "Datasheet" "" (id 3) (at 170.18 129.54 0)
-      (effects (font (size 1.27 1.27)) hide)
-    )
-    (pin "1")
-  )
   (symbol (lib_id "power:GND") (at 45.72 22.86 180) (unit 1)
     (in_bom yes) (on_board yes)
@@
       (reference "#PWR041") (unit 1) (value "GND") (footprint "")
     )
-    (path "/ed698bcb-0c1c-4ad0-868f-65e0c2a35d5b"
-      (reference "#PWR042") (unit 1) (value "GND") (footprint "")
-    )
     (path "/81e90d3c-0e7e-4548-aaef-76f2edbb33ef"
       (reference "#PWR043") (unit 1) (value "GND") (footprint "")
@@
       (reference "J11") (unit 1) (value "Conn_01x03_MountingPin") (footprint "Connector_JST:JST_SH_BM03B-SRSS-TB_1x03-1MP_P1.00mm_Vertical")
     )
-    (path "/6df9a874-ecd0-4b3b-8197-f1681d0f3dcc"
-      (reference "J12") (unit 1) (value "Conn_01x02") (footprint "Connector_PinSocket_2.54mm:PinSocket_1x02_P2.54mm_Vertical")
-    )
     (path "/b91526a1-4a34-4124-9d96-fa092757f2e9"
-      (reference "J13") (unit 1) (value "Conn_01x02") (footprint "Connector_AMASS:AMASS_XT30U-M_1x02_P5.0mm_Vertical")
+      (reference "J12") (unit 1) (value "Conn_01x02") (footprint "Connector_AMASS:AMASS_XT30U-M_1x02_P5.0mm_Vertical")
+    )
+    (path "/63dc45c8-991c-438d-a4b6-28fc5c714bfb"
+      (reference "J13") (unit 1) (value "Conn_01x01") (footprint "Connector_Wire:SolderWirePad_1x01_SMD_1x2mm")
     )
     (path "/50328183-6186-4e3a-ac46-25f88f890007"

Commit message: LegoRCHub_10ch: improved layout: beta-3
Other:
- title: (none) -> Lego RC Hub 10ch v1
Changed lines of the file:
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@@
 (kicad_sch (version 20211123) (generator eeschema)
   (paper "A4")
+  (title_block
+    (title "Lego RC Hub 10ch v1")
+  )
   (junction (at 237.871 148.59) (diameter 0) (color 0 0 0 0)
   )

Commit message: Lego RC Hub 10ch v2: fully migrated to KiCad8
Parts:
- U1, U2, U3, U4, U5, U6: footprint Package_SO:Texas_HTSOP-8-1EP_3.9x4.9mm_P1.27mm_EP2.95x4.9mm_Mask2.4x3.1mm_ThermalVias -> CustomFootprints:Texas_HTSOP-8-1EP_3.9x4.9mm_P1.27mm_EP2.95x4.9mm_Mask2.4x3.1mm_ThermalVias
Other:
- title: Lego RC Hub 10ch v1 -> Lego RC Hub 10ch v2

Commit message: Lego RC Hub 10ch v3: improved zones
Other:
- title: Lego RC Hub 10ch v2 -> Lego RC Hub 10ch v3
Changed lines of the file:
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@@
 	(paper "A4")
 	(title_block
-		(title "Lego RC Hub 10ch v2")
+		(title "Lego RC Hub 10ch v3")
 	)
 	(junction
