File: PCB/LegoRCHub_10ch/LegoRCHub_10ch.kicad_sch (KiCad schematic)
At the start: 43 parts, among them J1 Conn_01x02, J10 Conn_01x03, J11 Conn_01x03_MountingPin, J12 Conn_01x02, J13 Conn_01x01, J2 Conn_01x02, J3 Conn_01x02, J4 Conn_01x02, J5 Conn_01x02, J6 Conn_01x02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

Commit message: PCB: working on double CPU design...
Parts:
- added C23: 100nF, Capacitor_SMD:C_1206_3216Metric_Pad1.33x1.80mm_HandSolder, symbol Device:C_Small
- added J14: Conn_01x01, Connector_Wire:SolderWirePad_1x01_SMD_1x2mm, symbol Connector_Generic:Conn_01x01
- added U9: ATtiny3226-X, Package_SO:SSOP-20_5.3x7.2mm_P0.65mm, symbol MCU_Microchip_ATtiny:ATtiny3226-X
Connections:
- net GND: now also C23.1, U9.20 (GND)
- net IBus: now also U9.8 (PB3)
- net VCC: now also C23.2, U9.1 (VCC)
- new net UPDI_2: J14.1 (Pin_1), U9.16 (~{RESET}/PA0)
Other:
- moved on the sheet: C13, C16, J12, U7
